File: LrTMAX.kicad_sch (KiCad schematic)
At the start: 126 parts, among them J1 USB_C_Receptacle_USB2.0, J2 Conn_02x05_Odd_Even, Q1 2N7002, SW1 Tact_SW_8mm, SW10 EC11_SMD, SW11 EC11_SMD, SW12 EC11_SMD, SW13 EC11_SMD, SW14 EC11_SMD, SW15 EC11_SMD, SW16 EC11_SMD, SW17 EC11_SMD, SW2 Tact_SW_8mm, SW20 SW_SPST, SW3 Tact_SW_8mm, SW4 Tact_SW_8mm, SW5 Tact_SW_8mm, SW6 Tact_SW_8mm, SW7 Tact_SW_8mm, SW8 Tact_SW_8mm, U1 STM32F072C8Tx, U3 SSD1306_OLED_0.91, U4 SPX3819M5-L3-3TR

Commit message: trace drawn except CPU.
Connections:
- net DFU: now reaches R7.2, SW20.2 (B), U1.44 (BOOT0)
Changed lines of the file:
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@@
+    (effects (font (size 1.27 1.27)) (justify left bottom))
+  )
+  (label "DFU" (at 185.42 72.39 0)
     (effects (font (size 1.27 1.27)) (justify left bottom))
   )
